File: experiments/polymodnano/modulepcb/modulepcb.kicad_pcb (KiCad board)
At the start: 2 copper layers, 40.3 x 128.5 mm, 23 parts, among them J1 Conn_01x15_Female, J2 Conn_01x01_Male, J3 Conn_01x01_Male, J4 Conn_01x15_Female, J5 Conn_01x08_Male, J6 Conn_01x08_Male, J7 Conn_01x04_Female, J8 Conn_01x04_Female, SW1 SW_Push, SW2 SW_SPDT

Commit message: pcb done
Routing:
- net +5V: track 0.00 -> 187.9 mm
- net /POT2: track 0.00 -> 87.4 mm
- net /POT1: track 0.00 -> 79.6 mm
- net /POT4: track 0.00 -> 70.4 mm
- net /LED1: track 0.00 -> 67.4 mm
- net /ID: track 0.00 -> 65.8 mm
- net /POT3: track 0.00 -> 65.6 mm
- net /POT6: track 0.00 -> 59.3 mm
- net /POT5: track 0.00 -> 57.6 mm
- net /LED2: track 0.00 -> 53.8 mm
- net /SCL: track 0.00 -> 36.5 mm
- net /SDA: track 0.00 -> 34.5 mm
- net /RESET: track 0.00 -> 20.3 mm
- net /OUT4: track 0.00 -> 19.1 mm
- net /OUT1: track 0.00 -> 19.1 mm
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- added copper zone on B.Cu, net GND
- added copper zone on F.Cu, net GND
